File: schematic.kicad_pcb (KiCad board)
At the start: 2 copper layers, 165.7 x 122.2 mm, 81 parts, among them J3 USB_C_Receptacle_USB2.0_16P

Commit message: Add mounting holes and TVS diodes
Parts:
- added D26: ESD5Z5.0C, Diode_SMD:D_SOD-523, F.Cu at (171.1, 109.7)
- added D27: ESD5Z5.0C, Diode_SMD:D_SOD-523, F.Cu at (168.9, 116.1)
- added D28: ESD5Z5.0C, Diode_SMD:D_SOD-523, F.Cu at (167.1, 124.2)
- added D29: ESD5Z5.0C, Diode_SMD:D_SOD-523, F.Cu at (189.0, 137.1)
- added D30: ESD5Z5.0C, Diode_SMD:D_SOD-523, F.Cu at (187.8, 138.2)
- added D31: ESD5Z5.0C, Diode_SMD:D_SOD-523, F.Cu at (187.8, 143.2)
- added D32: ESD5Z5.0C, Diode_SMD:D_SOD-523, F.Cu at (187.2, 146.0)
- added D33: ESD5Z5.0C, Diode_SMD:D_SOD-523, F.Cu at (186.8, 148.8)
- added D34: ESD5Z5.0C, Diode_SMD:D_SOD-523, F.Cu at (165.6, 135.7)
- added D35: ESD5Z5.0C, Diode_SMD:D_SOD-523, F.Cu at (166.3, 146.5)
- added D36: ESD5Z5.0C, Diode_SMD:D_SOD-523, F.Cu at (179.2, 148.8)
- added D37: ESD5Z5.0C, Diode_SMD:D_SOD-523, F.Cu at (165.2, 139.0)
- added D38: ESD5Z5.0C, Diode_SMD:D_SOD-523, F.Cu at (166.4, 131.9)
- added D39: ESD5Z5.0C, Diode_SMD:D_SOD-523, F.Cu at (164.9, 131.6)
- added D40: ESD5Z5.0C, Diode_SMD:D_SOD-523, F.Cu at (162.9, 130.1)
- added D41: ESD5Z5.0C, Diode_SMD:D_SOD-523, F.Cu at (166.9, 119.8)
- added D42: ESD5Z5.0C, Diode_SMD:D_SOD-523, F.Cu at (179.7, 117.4)
- added JP2: SolderJumper_2_Bridged, Jumper:SolderJumper-2_P1.3mm_Bridged_RoundedPad1.0x1.5mm, F.Cu at (113.8, 132.2)
- added MH1: MountingHole_Pad, MountingHole:MountingHole_3mm_Pad_Via, F.Cu at (184.5, 109.5)
- added MH2: MountingHole_Pad, MountingHole:MountingHole_3mm_Pad_Via, F.Cu at (133.6, 78.4)
- added MH3: MountingHole_Pad, MountingHole:MountingHole_3mm_Pad_Via, F.Cu at (188.0, 184.2)
- added MH4: MountingHole_Pad, MountingHole:MountingHole_3mm_Pad_Via, F.Cu at (73.0, 163.8)
- added MH5: MountingHole_Pad, MountingHole:MountingHole_3mm_Pad_Via, F.Cu at (146.2, 182.5)
- added MH6: MountingHole_Pad, MountingHole:MountingHole_3mm_Pad_Via, F.Cu at (67.2, 98.2)
- added MH_GND1: MountingHole_Pad, MountingHole:MountingHole_3mm_Pad_Via, F.Cu at (120.0, 132.3)
Connections:
- net /NC renamed /NC_2
- net /P15 renamed /P22
- net /P16 renamed /P23
- net /P18 renamed /P26
- net /P19 renamed /P27
- net /P3 renamed /HAND
- D1 pad 1: /P20 -> /P28
- D10 pad 1: /P20 -> /P28
- D11 pad 1: /P2 -> /P29
- D12 pad 1: /P1 -> /P0
- D13 pad 1: /P20 -> /P28
- D14 pad 1: /P2 -> /P29
- D15 pad 1: /P1 -> /P0
- D16 pad 1: /P20 -> /P28
- D17 pad 1: /P2 -> /P29
- D18 pad 1: /P1 -> /P0
- D19 pad 1: /P8 -> /P9
- D2 pad 1: /P2 -> /P29
- D20 pad 1: /P14 -> /P21
- D21 pad 1: /P8 -> /P9
- D22 pad 1: /P14 -> /P21
- D23 pad 1: /P8 -> /P9
- D24 pad 1: /P8 -> /P9
- D25 pad 1: /P8 -> /P9
- D3 pad 1: /P1 -> /P0
- D4 pad 1: /P20 -> /P28
- D5 pad 1: /P2 -> /P29
- D6 pad 1: /P1 -> /P0
- D7 pad 1: /P20 -> /P28
- D8 pad 1: /P2 -> /P29
- D9 pad 1: /P1 -> /P0
- J3 pad A5: unconnected-(J3-CC1-PadA5) -> GND
- J3 pad A8: unconnected-(J3-SBU1-PadA8) -> GND
- J3 pad B5: unconnected-(J3-CC2-PadB5) -> GND
- J3 pad B8: unconnected-(J3-SBU2-PadB8) -> GND
- LED12 pad 2: /LED23 -> /LED22
- LED12 pad 4: /LED22 -> /LED21
- LED15 pad 2: /LED22 -> /LED21
- LED15 pad 4: /LED21 -> /LED20
- LED18 pad 2: /LED21 -> /LED20
- LED25 pad 4: /P9 -> /LED
- LED3 pad 4: /LED25 -> /LED24
- LED6 pad 2: /LED25 -> /LED24
- LED6 pad 4: /LED24 -> /LED23
- LED9 pad 2: /LED24 -> /LED23
- LED9 pad 4: /LED23 -> /LED22
- S1 pad 1: /P10 -> /P20
- S13 pad 1: /P21 -> /P2
- S14 pad 1: /P21 -> /P2
- S15 pad 1: /P21 -> /P2
- S16 pad 1: /P0 -> /P1
- S17 pad 1: /P0 -> /P1
- S18 pad 1: /P0 -> /P1
- S2 pad 1: /P10 -> /P20
- S21 pad 1: /P21 -> /P2
- S22 pad 1: /P21 -> /P2
- S23 pad 1: /P0 -> /P1
- S3 pad 1: /P10 -> /P20
- U1 pad 0: /P1 -> /P0
- U1 pad 1: /P0 -> /P1
- U1 pad 10: unconnected-(U1-GP10-Pad10) -> /NC2
- U1 pad 11: unconnected-(U1-GP11-Pad11) -> /NC1
- U1 pad 2: /P21 -> /P2
- U1 pad 20: /P10 -> /P20
- U1 pad 21: /P14 -> /P21
- U1 pad 28: /P20 -> /P28
- U1 pad 29: /P2 -> /P29
- U1 pad 4: unconnected-(U1-GP4-Pad4) -> /NC3
- U1 pad 8: /P9 -> /LED
- U1 pad 9: /P8 -> /P9
Routing:
- net /P10: track 235.5 -> 0.00 mm, vias 5 -> 0
- net /P29: track 0.00 -> 204.6 mm
- net /P28: track 0.00 -> 190.7 mm
- net /P8: track 146.8 -> 0.00 mm
- net /P21: track 228.7 -> 90.7 mm, vias 5 -> 0
- net /P9: track 53.9 -> 146.8 mm, vias 1 -> 0
- net /P14: track 90.7 -> 0.00 mm
- net Vraw: track 942.4 -> 872.5 mm
- net /LED: track 0.00 -> 53.9 mm, vias 0 -> 1
- net GND: track 986.5 -> 935.3 mm, vias 138 -> 148
- net /P20: track 190.7 -> 235.5 mm, vias 0 -> 5
- net /LED25: track 26.8 -> 0.00 mm, vias 2 -> 0
- net /LED20: track 0.00 -> 25.8 mm, vias 0 -> 2
- net /P2: track 204.6 -> 228.7 mm, vias 0 -> 5
- net /P1: track 208.2 -> 186.3 mm, vias 0 -> 4
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